File: pcb/ipotcas/ipotcas.kicad_sch (KiCad schematic)
At the start: 74 parts, among them J1 Screw_Terminal_01x02, J10 Conn_01x03, J11 AudioJack4, J12 Conn_01x07, J13 Conn_01x03, J14 Conn_01x02, J2 Screw_Terminal_01x02, J3 Screw_Terminal_01x02, J4 Conn_01x06, J5 Barrel_Jack_Switch, J6 AudioJack4, J7 Conn_01x03, J8 Conn_01x03, J9 Conn_01x02, U1 NUCLEO144-F767ZI, U2 MCP602, U3 LM741, U4 TC7662Bx0A, Y1 SG-210STF

Commit message: Port RX to new PCB
Parts:
- C1, C10, C12, C13, C19, C2, C22, C23, C5, C6, C7, C8, C9: JLC P/N (none) -> C1525
- C14, C15, C16, C17, C18, C20, C21, C24: JLC P/N (none) -> C16780
- C3, C4: JLC P/N (none) -> C15525
- D1: footprint LED_SMD:LED_0603_1608Metric -> LED_SMD:LED_0805_2012Metric_Pad1.15x1.40mm_HandSolder; JLC P/N (none) -> C2287
- D2: footprint LED_SMD:LED_0603_1608Metric -> LED_SMD:LED_0805_2012Metric_Pad1.15x1.40mm_HandSolder; JLC P/N (none) -> C12624
- D3, D5: footprint LED_SMD:LED_0603_1608Metric -> LED_SMD:LED_0805_2012Metric_Pad1.15x1.40mm_HandSolder; JLC P/N (none) -> C2290
- D4: footprint LED_SMD:LED_0603_1608Metric -> LED_SMD:LED_0805_2012Metric_Pad1.15x1.40mm_HandSolder; JLC P/N (none) -> C2286
- J1, J2, J3: JLC P/N (none) -> C592976
- J11, J6: JLC P/N (none) -> C431535
- R1: JLC P/N (none) -> C11702
- R10, R12: JLC P/N (none) -> C25562
- R11, R7, R8, R9: JLC P/N (none) -> C25092
- R15, R16: footprint Capacitor_SMD:C_0402_1005Metric -> Resistor_SMD:R_0402_1005Metric; JLC P/N (none) -> C11702
- R2, R5: JLC P/N (none) -> C25900
- R27, R30: JLC P/N (none) -> C25546
- R28: JLC P/N (none) -> C25744
- R29: footprint Resistor_SMD:R_0603_1608Metric_Pad0.98x0.95mm_HandSolder -> Resistor_SMD:R_0402_1005Metric; JLC P/N (none) -> C25879
- R3: JLC P/N (none) -> C118954
- R4: JLC P/N (none) -> C25768
- R6: JLC P/N (none) -> C25077
- U2: JLC P/N (none) -> C360037
- U3: JLC P/N (none) -> C5145278
- U4: JLC P/N (none) -> C81518
- U5: JLC P/N (none) -> C24109
- Y1: JLC P/N (none) -> C255992
Connections:
- net GND: no longer C10.2, C11.2, C12.2, C19.2, C2.2, C22.2, C4.2, C5.2, C8.2, C9.2, J1.1 (Pin_1), J10.1 (Pin_1), J11.R2, J14.2 (Pin_2), J2.1 (Pin_1), J3.1 (Pin_1), J5.2, J6.R2, J7.2 (Pin_2), J8.2 (Pin_2), J9.1 (Pin_1), R10.2, R12.2, U1.104 (AGND), U2.4 (V-), U3.2 (-), U4.3 (GND), U5.17 (AV_{SS})
- new net GNDA: C10.2, C11.2, C12.2, C19.2, C2.2, C22.2, C4.2, C5.2, C8.2, C9.2, J1.1 (Pin_1), J10.1 (Pin_1), J11.R2, J14.2 (Pin_2), J2.1 (Pin_1), J3.1 (Pin_1), J5.2, J6.R2, J7.2 (Pin_2), J8.2 (Pin_2), J9.1 (Pin_1), R10.2, R12.2, U1.104 (AGND), U2.4 (V-), U3.2 (-), U4.3 (GND), U5.17 (AV_{SS})
